Commit message: feat: sync latest workspace source changes
Co-Authored-By: Claude Opus 4.8 <noreply@anthropic.com>

File: src/gantry_robot_moveit_config_sim/config/gantry_robot.ros2_control.xacro (robot description, xacro)
@@ -15,4 +15,11 @@
                 <state_interface name="velocity"/>
             </joint>
+            <!-- <joint name="y_rail_joint">
+                <command_interface name="position"/>
+                <state_interface name="position">
+                  <param name="initial_value">${initial_positions['y_rail_joint']}</param>
+                </state_interface>
+                <state_interface name="velocity"/>
+            </joint> -->
             <joint name="joint_1_2">
                 <command_interface name="position"/>

File: src/models/urdf/gantry_robot.xacro (robot description, xacro)
@@ -6,4 +6,24 @@
   </material>
   <!-- link name="world" / -->
+  <link name="floor">
+    <visual>
+      <origin xyz="0 0 0" rpy="0 0 0" />
+      <geometry>
+        <box size="2 2 0.01" />
+      </geometry>
+      <material name="grey" />
+    </visual>
+    <collision>
+      <origin xyz="0 0 0" rpy="0 0 0" />
+      <geometry>
+        <box size="2 2 0.01" />
+      </geometry>
+    </collision>
+  </link>
+  <joint name="world_to_floor" type="fixed">
+    <parent link="world" />
+    <child link="floor" />
+    <origin xyz="0 0 -0.006" rpy="0 0 0" />
+  </joint>
   <!-- IPM (Imaginary Point Marker) - 参考点 -->
   <link name="ipm">
@@ -26,5 +46,5 @@
     <parent link="world" />
     <child link="ipm" />
-    <origin xyz="0.5 -0.2 0.6" rpy="1.57 0 -1.57" />
+    <origin xyz="0.0 0.0 0.0" rpy="1.57 0 -1.57" />
   </joint>
   <link name="x_rail">
@@ -37,8 +57,21 @@
     <parent link="world" />
     <child link="x_rail" />
+    <origin xyz="-0.2 0 0" rpy="0 0 0" />
+    <axis xyz="1 0 0"/>
+    <limit lower="-0.4" upper="0.2" velocity="0.5" effort="1000"/>
+  </joint>
+  <!-- <link name="y_rail">
+    <inertial>
+      <mass value="5.0" />
+      <inertia ixx="0.1" ixy="0.0" ixz="0.0" iyy="0.1" iyz="0.0" izz="0.1" />
+    </inertial>
+  </link>
+  <joint name="y_rail_joint" type="prismatic">
+    <parent link="x_rail" />
+    <child link="y_rail" />
     <origin xyz="0 0 0" rpy="0 0 0" />
-    <axis xyz="1 0 0"/>
-    <limit lower="0" upper="0.15" velocity="0.5" effort="1000"/>
-  </joint>
+    <axis xyz="0 1 0"/>
+    <limit lower="-0.0" upper="0.0" velocity="0.5" effort="1000"/>
+  </joint> -->
   <link name="link1">
     <visual>
@@ -63,5 +96,5 @@
     <parent link="x_rail" />
     <child link="link1" />
-    <origin xyz="0 0 0.35" rpy="0 0 0" />
+    <origin xyz="-0.1 0.0 0.35" rpy="0 0 0" />
   </joint>
   <link name="link2">
